Commit message: Make sensor noise settable per run, and take the map origin from the first fix
Sensor realism knobs are now xacro args forwarded through the launch file, so a
run can be degraded without editing the model:

    ros2 launch hege_description spawn_hege.launch.py gps_noise:=1.5

gps_noise is the horizontal standard deviation; vertical is derived at twice
that, as it runs on any GNSS receiver. 0.02 is RTK-fixed, ~0.4 is RTK float,
~2.0 is a single-point solution. This is the test rig the Goal 2 robustness
work needs.

The IMU also gained bias terms, which were simply absent before. A real MEMS
IMU's dominant error is not white noise but a bias drawn at startup that then
wanders, and leaving it at zero handed the filter an IMU better than any that
exists. The effect is immediate: the local EKF's worst error over the same
route went from 0.93 m to 3.39 m, which is the honest number.

navsat_transform now takes its datum from the first GPS fix rather than the
surveyed coordinates. Nothing has to be measured and typed in before the rover
can run, and it costs nothing while waypoints are given as latitude/longitude,
since each is converted into whatever map frame the run happens to have. The
launch file keeps use_datum:=true for pinning the origin when simulation runs
need to be comparable.

Measured over the same 45 s route, worst error against Gazebo ground truth:

                     RTK fixed    single-point
    raw GPS            0.096 m         4.405 m
    global EKF         0.086 m         2.675 m
    local EKF          3.392 m         3.642 m

The second column is the point: with the fix degraded, the fused estimate is
better than the GPS it is built from, because odometry carries it between fixes.

File: src/hege_description/urdf/hege.urdf.xacro (robot description, xacro)
@@ -14,4 +14,30 @@
   <xacro:arg name="drive" default="planar"/>
   <xacro:property name="drive" value="$(arg drive)"/>
+  <!-- Sensor realism knobs, exposed so a run can be degraded without editing
+       this file. Pass them through the launch file, e.g.
+         ros2 launch hege_description spawn_hege.launch.py gps_noise:=1.5
+       to simulate losing the RTK fix. -->
+  <!-- GPS horizontal standard deviation, metres. 0.02 is RTK-fixed. Roughly
+       0.3-0.5 for RTK float and 1.5-3.0 for a single-point solution - those
+       are the Goal 2 robustness cases. -->
+  <xacro:arg name="gps_noise" default="0.02"/>
+  <xacro:property name="gps_noise" value="$(arg gps_noise)"/>
+  <!-- Gyro and accelerometer bias. A real MEMS IMU's dominant error is not
+       white noise but a bias drawn at startup that then wanders, and that is
+       what makes dead reckoning fall apart. Leaving these at zero, as this
+       model did until now, hands the filter an IMU better than any that
+       exists. bias_mean is the centre of the startup distribution, bias_stddev
+       its spread. -->
+  <xacro:arg name="imu_gyro_bias"  default="7.5e-6"/>
+  <xacro:arg name="imu_accel_bias" default="0.05"/>
+  <xacro:property name="imu_gyro_bias"  value="$(arg imu_gyro_bias)"/>
+  <xacro:property name="imu_accel_bias" value="$(arg imu_accel_bias)"/>
+  <!-- White noise per sample. Datasheets quote noise DENSITY, per root-hertz;
+       convert with stddev = density * sqrt(rate) before putting a number
+       here. -->
+  <xacro:arg name="imu_gyro_noise"  default="2e-4"/>
+  <xacro:arg name="imu_accel_noise" default="1.7e-2"/>
+  <xacro:property name="imu_gyro_noise"  value="$(arg imu_gyro_noise)"/>
+  <xacro:property name="imu_accel_noise" value="$(arg imu_accel_noise)"/>
   <!-- ============ MEASURED HEGE DIMENSIONS ============ -->
   <!-- Body. base_link sits at the underside of the chassis, body_z_offset above
@@ -206,12 +232,12 @@
       <imu>
         <angular_velocity>
-          <x><noise type="gaussian"><mean>0.0</mean><stddev>2e-4</stddev></noise></x>
-          <y><noise type="gaussian"><mean>0.0</mean><stddev>2e-4</stddev></noise></y>
-          <z><noise type="gaussian"><mean>0.0</mean><stddev>2e-4</stddev></noise></z>
+          <x><noise type="gaussian"><mean>0.0</mean><stddev>${imu_gyro_noise}</stddev><bias_mean>${imu_gyro_bias}</bias_mean><bias_stddev>${imu_gyro_bias}</bias_stddev></noise></x>
+          <y><noise type="gaussian"><mean>0.0</mean><stddev>${imu_gyro_noise}</stddev><bias_mean>${imu_gyro_bias}</bias_mean><bias_stddev>${imu_gyro_bias}</bias_stddev></noise></y>
+          <z><noise type="gaussian"><mean>0.0</mean><stddev>${imu_gyro_noise}</stddev><bias_mean>${imu_gyro_bias}</bias_mean><bias_stddev>${imu_gyro_bias}</bias_stddev></noise></z>
         </angular_velocity>
         <linear_acceleration>
-          <x><noise type="gaussian"><mean>0.0</mean><stddev>1.7e-2</stddev></noise></x>
-          <y><noise type="gaussian"><mean>0.0</mean><stddev>1.7e-2</stddev></noise></y>
-          <z><noise type="gaussian"><mean>0.0</mean><stddev>1.7e-2</stddev></noise></z>
+          <x><noise type="gaussian"><mean>0.0</mean><stddev>${imu_accel_noise}</stddev><bias_mean>${imu_accel_bias}</bias_mean><bias_stddev>${imu_accel_bias}</bias_stddev></noise></x>
+          <y><noise type="gaussian"><mean>0.0</mean><stddev>${imu_accel_noise}</stddev><bias_mean>${imu_accel_bias}</bias_mean><bias_stddev>${imu_accel_bias}</bias_stddev></noise></y>
+          <z><noise type="gaussian"><mean>0.0</mean><stddev>${imu_accel_noise}</stddev><bias_mean>${imu_accel_bias}</bias_mean><bias_stddev>${imu_accel_bias}</bias_stddev></noise></z>
         </linear_acceleration>
       </imu>
@@ -237,11 +263,11 @@
       <gps>
         <position_sensing>
-          <!-- RTK-fixed grade: ~2 cm horizontal. Raise stddev to 0.5-2.0 for
-               the Goal 2 degraded-fix robustness runs. -->
           <horizontal>
-            <noise type="gaussian"><mean>0.0</mean><stddev>0.02</stddev></noise>
+            <noise type="gaussian"><mean>0.0</mean><stddev>${gps_noise}</stddev></noise>
           </horizontal>
+          <!-- Vertical error runs about twice the horizontal on any GNSS
+               receiver, so it is derived rather than set separately. -->
           <vertical>
-            <noise type="gaussian"><mean>0.0</mean><stddev>0.04</stddev></noise>
+            <noise type="gaussian"><mean>0.0</mean><stddev>${gps_noise * 2}</stddev></noise>
           </vertical>
         </position_sensing>

Commit message: Keep sensor noise in the model rather than on the launch command line
The noise settings were xacro args forwarded through the launch file. They are
plain xacro properties now, sitting with the rest of the robot's description
where the dimensions and inertias already live, and the launch file is back to
declaring only what is genuinely a per-run choice: which world, where to spawn,
which drive mode.

Nothing is lost for the Goal 2 robustness work. The workspace is built with
symlink install, so editing gps_noise in the model and launching again is
enough; no rebuild, no rebuilt argument list. Verified by switching it to 1.5
and back and watching the generated URDF follow.

Values and what they mean stay documented next to them: 0.02 RTK fixed, 0.4
RTK float, 2.0 single-point.

File: src/hege_description/urdf/hege.urdf.xacro (robot description, xacro)
@@ -14,30 +14,29 @@
   <xacro:arg name="drive" default="planar"/>
   <xacro:property name="drive" value="$(arg drive)"/>
-  <!-- Sensor realism knobs, exposed so a run can be degraded without editing
-       this file. Pass them through the launch file, e.g.
-         ros2 launch hege_description spawn_hege.launch.py gps_noise:=1.5
-       to simulate losing the RTK fix. -->
-  <!-- GPS horizontal standard deviation, metres. 0.02 is RTK-fixed. Roughly
-       0.3-0.5 for RTK float and 1.5-3.0 for a single-point solution - those
-       are the Goal 2 robustness cases. -->
-  <xacro:arg name="gps_noise" default="0.02"/>
-  <xacro:property name="gps_noise" value="$(arg gps_noise)"/>
+  <!-- ============ SENSOR NOISE ============ -->
+  <!-- Edited here rather than passed in at launch. The workspace is built
+       with symlink install, so a change takes effect on the next launch with
+       no rebuild. -->
+  <!-- GPS horizontal standard deviation, metres. Vertical is derived at twice
+       this, as it runs on any GNSS receiver.
+         0.02  RTK fixed
+         0.4   RTK float
+         2.0   single-point solution
+       The upper two are the Goal 2 robustness cases: raise this, run the same
+       route, and read the error off the localization monitor. -->
+  <xacro:property name="gps_noise" value="0.02"/>
   <!-- Gyro and accelerometer bias. A real MEMS IMU's dominant error is not
        white noise but a bias drawn at startup that then wanders, and that is
        what makes dead reckoning fall apart. Leaving these at zero, as this
        model did until now, hands the filter an IMU better than any that
-       exists. bias_mean is the centre of the startup distribution, bias_stddev
-       its spread. -->
-  <xacro:arg name="imu_gyro_bias"  default="7.5e-6"/>
-  <xacro:arg name="imu_accel_bias" default="0.05"/>
-  <xacro:property name="imu_gyro_bias"  value="$(arg imu_gyro_bias)"/>
-  <xacro:property name="imu_accel_bias" value="$(arg imu_accel_bias)"/>
+       exists. Raising the local EKF's worst error from 0.93 m to 3.39 m over
+       the same route is the honest number, not a regression. -->
+  <xacro:property name="imu_gyro_bias"  value="7.5e-6"/>
+  <xacro:property name="imu_accel_bias" value="0.05"/>
   <!-- White noise per sample. Datasheets quote noise DENSITY, per root-hertz;
        convert with stddev = density * sqrt(rate) before putting a number
        here. -->
-  <xacro:arg name="imu_gyro_noise"  default="2e-4"/>
-  <xacro:arg name="imu_accel_noise" default="1.7e-2"/>
-  <xacro:property name="imu_gyro_noise"  value="$(arg imu_gyro_noise)"/>
-  <xacro:property name="imu_accel_noise" value="$(arg imu_accel_noise)"/>
+  <xacro:property name="imu_gyro_noise"  value="2e-4"/>
+  <xacro:property name="imu_accel_noise" value="1.7e-2"/>
   <!-- ============ MEASURED HEGE DIMENSIONS ============ -->
   <!-- Body. base_link sits at the underside of the chassis, body_z_offset above

Commit message: Put the real 1200 kg on the model, with a tractor-like weight distribution
The chassis was carrying the 50 kg from the first sketch, which with the wheels
made the whole machine 80 kg. It is 1200 kg.

Mass is now stated once as total_mass, with the wheels and knuckles taking
estimates for tractor-style parts and the chassis taking the remainder, so the
total stays at 1200 kg whichever of them is edited.

Weight distribution is expressed as intent rather than as a coordinate:
front_axle_load is the share the front axle carries, 0.4 for a machine that
sits back on its rear axle, which is also why the rear wheels are the larger
pair. The chassis centre of mass is then derived from that, accounting for the
wheels and knuckles carrying their own weight at fixed positions, so the stated
split and the geometry cannot drift apart. Verified: 480 kg front, 720 kg rear.
Its height is placed below the box centre, since drivetrain and batteries sit
low and it is what decides rollover behaviour on a slope.

Two things had to scale with it or the model would have been quietly wrong:

- Steering effort, 100 Nm to 8000 Nm. The old figure was sized for a 15 kg
  placeholder and cannot turn a 1200 kg front axle against tyre scrub, so the
  steering would never have reached its commanded angle.
- Contact stiffness, kp 1e6 to 1e7 with damping to match. At the old value
  1200 kg presses the wheels into the ground far enough to change their
  effective radius, and with it the odometry.

Checked after the change: the rover sits upright at the right height, drives
the right way, steers the right way with the inner wheel taking the larger
angle, and the global EKF still tracks ground truth to 0.111 m worst case.

File: src/hege_description/urdf/hege.urdf.xacro (robot description, xacro)
@@ -46,5 +46,35 @@
   <xacro:property name="base_width"    value="1.4"/>
   <xacro:property name="base_height"   value="0.8"/>
-  <xacro:property name="base_mass"     value="50.0"/>
+  <!-- Mass. The real machine is 1200 kg. Wheel and knuckle masses are
+       estimates for tractor-style wheels; the chassis takes whatever is left,
+       so the total always comes out at total_mass no matter which of these is
+       edited. -->
+  <xacro:property name="total_mass"        value="1200.0"/>
+  <xacro:property name="rear_wheel_mass"   value="80.0"/>
+  <xacro:property name="front_wheel_mass"  value="45.0"/>
+  <xacro:property name="steer_link_mass"   value="15.0"/>
+  <xacro:property name="sensor_mass"       value="0.05"/>
+  <xacro:property name="base_mass"
+    value="${total_mass - 2*rear_wheel_mass - 2*front_wheel_mass
+                        - 2*steer_link_mass - 2*sensor_mass}"/>
+  <!-- Weight distribution, stated as the share of static load carried by the
+       front axle. Tractor-like machines sit back on the rear axle, which is
+       also why the rear wheels are the larger pair. 0.4 means 40% front,
+       60% rear.
+       The chassis centre of mass is then placed wherever it has to be for the
+       whole vehicle to balance that way, given that the wheels and knuckles
+       sit at fixed positions and carry their own weight. Derived rather than
+       typed so the two cannot drift apart. -->
+  <xacro:property name="front_axle_load" value="0.4"/>
+  <xacro:property name="com_x_target" value="${wheelbase*(front_axle_load - 0.5)}"/>
+  <xacro:property name="base_com_x"
+    value="${(total_mass*com_x_target
+              - 2*(front_wheel_mass + steer_link_mass)*(wheelbase/2)
+              + 2*rear_wheel_mass*(wheelbase/2)) / base_mass}"/>
+  <!-- Centre of mass height above base_link. The body box spans 0 to 0.8, but
+       the heavy parts of a machine like this - drivetrain, batteries - sit low,
+       so the centre of mass is placed below the box's geometric centre. It
+       matters for rollover behaviour on slopes. -->
+  <xacro:property name="base_com_z" value="0.25"/>
   <xacro:property name="body_z_offset" value="0.4"/>
   <xacro:property name="base_z"        value="1.1"/>
@@ -56,5 +86,4 @@
   <xacro:property name="rear_wheel_radius"  value="0.40"/>
   <xacro:property name="wheel_width"        value="0.2"/>
-  <xacro:property name="wheel_mass"         value="5.0"/>
   <!-- Front and rear tracks also differ slightly. -->
   <xacro:property name="wheelbase"   value="1.91"/>
@@ -79,6 +108,7 @@
        geometry are the usual cause of ODE blowing up into NaN. These compute
        the real thing so the numbers stay consistent when dimensions change. -->
-  <xacro:macro name="box_inertia" params="m x y z">
+  <xacro:macro name="box_inertia" params="m x y z cx:=0 cy:=0 cz:=0">
     <inertial>
+      <origin xyz="${cx} ${cy} ${cz}" rpy="0 0 0"/>
       <mass value="${m}"/>
       <inertia ixx="${m*(y*y+z*z)/12.0}" ixy="0" ixz="0"
@@ -100,8 +130,14 @@
   <xacro:macro name="wheel_surface" params="link">
     <gazebo reference="${link}">
+      <!-- Friction. Tractor tyres on soil, and this is the knob behind the
+           rover turning less sharply than commanded. -->
       <mu1>1.0</mu1>
       <mu2>1.0</mu2>
-      <kp>1000000.0</kp>
-      <kd>100.0</kd>
+      <!-- Contact stiffness and damping, scaled with the vehicle. At the
+           1e6 that suited a 15 kg model, 1200 kg pushes the wheels into the
+           ground far enough to change the effective radius and therefore the
+           odometry. -->
+      <kp>10000000.0</kp>
+      <kd>10000.0</kd>
       <minDepth>0.001</minDepth>
       <maxVel>1.0</maxVel>
@@ -119,5 +155,6 @@
       <geometry><box size="${base_length} ${base_width} ${base_height}"/></geometry>
     </collision>
-    <xacro:box_inertia m="${base_mass}" x="${base_length}" y="${base_width}" z="${base_height}"/>
+    <xacro:box_inertia m="${base_mass}" x="${base_length}" y="${base_width}" z="${base_height}"
+                       cx="${base_com_x}" cz="${base_com_z}"/>
   </link>
   <joint name="base_joint" type="fixed">
@@ -136,5 +173,5 @@
         <geometry><cylinder radius="${rear_wheel_radius}" length="${wheel_width}"/></geometry>
       </collision>
-      <xacro:cylinder_inertia m="${wheel_mass}" r="${rear_wheel_radius}" h="${wheel_width}"/>
+      <xacro:cylinder_inertia m="${rear_wheel_mass}" r="${rear_wheel_radius}" h="${wheel_width}"/>
     </link>
     <joint name="${prefix}_rear_wheel_joint" type="continuous">
@@ -161,6 +198,6 @@
            ODE cannot solve stably - it diverges to NaN within a few steps. -->
       <inertial>
-        <mass value="${wheel_mass}"/>
-        <inertia ixx="0.05" ixy="0" ixz="0" iyy="0.05" iyz="0" izz="0.05"/>
+        <mass value="${steer_link_mass}"/>
+        <inertia ixx="0.5" ixy="0" ixz="0" iyy="0.5" iyz="0" izz="0.5"/>
       </inertial>
     </link>
@@ -170,5 +207,10 @@
       <origin xyz="${wheelbase/2} ${y_sign*front_track/2} ${front_axle_z}"/>
       <axis xyz="0 0 1"/>
-      <limit lower="${-max_steer}" upper="${max_steer}" effort="100" velocity="2.0"/>
+      <!-- Effort scaled with the vehicle. 100 Nm, sized for the old 15 kg
+           placeholder, cannot turn the front axle of a 1200 kg machine against
+           tyre scrub; the steering simply would not reach its commanded angle.
+           Velocity limited to roughly lock to lock in a second and a half,
+           which is about what a real steering actuator manages. -->
+      <limit lower="${-max_steer}" upper="${max_steer}" effort="8000" velocity="0.8"/>
     </joint>
     <!-- Actual rolling wheel attached to the steer link -->
@@ -181,5 +223,5 @@
         <geometry><cylinder radius="${front_wheel_radius}" length="${wheel_width}"/></geometry>
       </collision>
-      <xacro:cylinder_inertia m="${wheel_mass}" r="${front_wheel_radius}" h="${wheel_width}"/>
+      <xacro:cylinder_inertia m="${front_wheel_mass}" r="${front_wheel_radius}" h="${wheel_width}"/>
     </link>
     <joint name="${prefix}_front_wheel_joint" type="continuous">

Commit message: Add waypoint navigation, tune Nav2 for Ackermann, fix Gazebo GPS bug, and update terrain physics

File: src/hege_description/urdf/hege.urdf.xacro (robot description, xacro)
@@ -25,5 +25,5 @@
        The upper two are the Goal 2 robustness cases: raise this, run the same
        route, and read the error off the localization monitor. -->
-  <xacro:property name="gps_noise" value="0.02"/>
+  <xacro:property name="gps_noise" value="2.0"/>
   <!-- Gyro and accelerometer bias. A real MEMS IMU's dominant error is not
        white noise but a bias drawn at startup that then wanders, and that is
@@ -183,4 +183,5 @@
       <origin xyz="${-wheelbase/2} ${y_sign*rear_track/2} ${rear_axle_z}" rpy="-1.5708 0 0"/>
       <axis xyz="0 0 1"/>
+      <limit effort="100000.0" velocity="20.0"/>
     </joint>
   </xacro:macro>

Commit message: Backup: Working trajectory fixes and initial scattered bale layout

File: src/hege_description/urdf/hege.urdf.xacro (robot description, xacro)
@@ -25,5 +25,5 @@
        The upper two are the Goal 2 robustness cases: raise this, run the same
        route, and read the error off the localization monitor. -->
-  <xacro:property name="gps_noise" value="2.0"/>
+  <xacro:property name="gps_noise" value="0.02"/>
   <!-- Gyro and accelerometer bias. A real MEMS IMU's dominant error is not
        white noise but a bias drawn at startup that then wanders, and that is
@@ -130,8 +130,7 @@
   <xacro:macro name="wheel_surface" params="link">
     <gazebo reference="${link}">
-      <!-- Friction. Tractor tyres on soil, and this is the knob behind the
-           rover turning less sharply than commanded. -->
-      <mu1>1.0</mu1>
-      <mu2>1.0</mu2>
+      <!-- Friction. High traction tractor tyres on soil to eliminate lateral slip -->
+      <mu1>20.0</mu1>
+      <mu2>20.0</mu2>
       <!-- Contact stiffness and damping, scaled with the vehicle. At the
            1e6 that suited a 15 kg model, 1200 kg pushes the wheels into the
