Commit message: fix(urdf): update robot dimensions and sensor offsets based on physical measurements

File: src/hege_description/urdf/hege.urdf.xacro (robot description, xacro)
@@ -45,5 +45,5 @@
   <xacro:property name="base_length"   value="2.2"/>
   <xacro:property name="base_width"    value="1.4"/>
-  <xacro:property name="base_height"   value="0.8"/>
+  <xacro:property name="base_height"   value="0.56"/>
   <!-- Mass. The real machine is 1200 kg. Wheel and knuckle masses are
        estimates for tractor-style wheels; the chassis takes whatever is left,
@@ -72,11 +72,12 @@
               - 2*(front_wheel_mass + steer_link_mass)*(wheelbase/2)
               + 2*rear_wheel_mass*(wheelbase/2)) / base_mass}"/>
-  <!-- Centre of mass height above base_link. The body box spans 0 to 0.8, but
+  <!-- Centre of mass height above base_link. The body box spans -0.28 to +0.28, but
        the heavy parts of a machine like this - drivetrain, batteries - sit low,
        so the centre of mass is placed below the box's geometric centre. It
        matters for rollover behaviour on slopes. -->
-  <xacro:property name="base_com_z" value="0.25"/>
-  <xacro:property name="body_z_offset" value="0.4"/>
-  <xacro:property name="base_z"        value="1.1"/>
+  <xacro:property name="base_com_z"    value="-0.05"/>
+  <xacro:property name="body_z_offset" value="0.0"/>
+  <xacro:property name="base_z"        value="1.10"/>
+  <xacro:property name="imu_z"         value="0.10"/>
   <!-- Front and rear wheels are DIFFERENT sizes on Hege: 27 cm front, 40 cm
        rear. Everything downstream has to respect that - the axle heights below
@@ -98,10 +99,7 @@
   <xacro:property name="front_axle_z" value="${front_wheel_radius - base_z}"/>
   <xacro:property name="rear_axle_z"  value="${rear_wheel_radius - base_z}"/>
-  <!-- GPS antenna height above base_link, as supplied. NOTE: the chassis box
-       spans 0 to 0.8 above base_link, so at 0.5 the antenna sits inside the
-       body volume. The real RTK antenna is mast-mounted above the roof; raise
-       this past base_height once the mast is measured, because
-       robot_localization uses base_link->gps_link as the lever arm. -->
-  <xacro:property name="gps_z" value="0.5"/>
+  <!-- GPS antenna height above base_link. Real measured height is 1.30 m from ground,
+       which is +0.20 m above base_link (1.10 m). -->
+  <xacro:property name="gps_z" value="0.20"/>
   <!-- ============ INERTIA HELPERS ============ -->
   <!-- Hand-written inertia tensors that disagree with the link's mass and
@@ -241,5 +239,5 @@
        the sensors still report in their own frame_name, which
        robot_state_publisher provides from the URDF. -->
-  <!-- IMU at the chassis centre -->
+  <!-- IMU at the Jetson / electronics enclosure (+0.10 m above base_link, 1.20 m from ground) -->
   <link name="imu_link">
     <inertial>
@@ -251,5 +249,5 @@
     <parent link="base_link"/>
     <child  link="imu_link"/>
-    <origin xyz="0 0 ${body_z_offset}" rpy="0 0 0"/>
+    <origin xyz="0 0 ${imu_z}" rpy="0 0 0"/>
   </joint>
   <!-- GPS antenna, top of chassis + mast -->

Commit message: Let PX4 SITL drive the Hege model
The two simulations never met. Ours plans and tracks a GPS route but drives
the rover through a Gazebo Classic Ackermann controller the real machine
does not have; the PX4 side proves the Pixhawk link but drives PX4's stock
0.321 m demo rover. This joins them, and leaves the Classic stack running
exactly as it was.

PX4 cannot use ros2_control or a URDF - it writes the joints itself over
gz-transport - so it needs an SDF model. Rather than hand-write a second
description that would drift from the first, hege.urdf.xacro grows a third
drive mode and the model is generated from it. The xacro stays the only
place the vehicle's geometry is written down.

Getting that model right is mostly about names PX4 does not let you
choose. GZBridge.cpp subscribes to four hardcoded topic paths, all under a
link called base_link, and a model that spells any of them differently
boots and looks healthy and never gives EKF2 that sensor. Worse,
URDF-to-SDF conversion lumps a fixed joint's child into its parent, so
base_link - base_footprint's fixed child - would have disappeared
entirely. Hence the preserved base_joint, and hence base_footprint
carrying a 1e-4 kg inertia in this mode and no other, since preserving the
joint makes it a real root link.

On the ROS side hege_localization and hege_navigation are included
unchanged; the whole difference is five launch arguments. Two needed
thought. There are no wheel encoders behind a Pixhawk, so ekf_local's
forward velocity comes from /px4/odom instead - position deliberately not,
since that is the same GPS navsat_transform already feeds in. And PX4's
offboard velocity branch drives forwards only, which the bridge enforces
by turning any negative linear.x into a stop, so the planner drops to
DUBIN, the controller loses allow_reversing, and the behaviour trees lose
the BackUp recovery they would otherwise hang on.

Verified here: all three drive modes expand cleanly with no
cross-contamination, the px4 URDF carries base_link and all four sensor
names, everything parses, 141 unit tests pass. Not verified: nothing has
been run. No Gazebo, no PX4 and no ROS in this environment, so model.sdf
has never been generated, the launch files are syntax-checked only, and
the airframe numbers are derived from the geometry rather than measured.
docs/px4_sitl.md says so plainly and lists what to suspect first.

File: src/hege_description/urdf/hege.urdf.xacro (robot description, xacro)
@@ -11,5 +11,15 @@
                          Real Ackermann kinematics, and the path to the real
                          robot, but currently held up by a controller bug that
-                         makes the rover creep at 1 m/s on startup. -->
+                         makes the rover creep at 1 m/s on startup.
+         px4           - Gazebo Harmonic, driven by PX4 SITL rather than by
+                         ROS. Nothing in this mode talks to ROS at all: PX4's
+                         gz_bridge reads the sensors and writes the wheel and
+                         steering joints over gz-transport, and ROS only sees
+                         the vehicle through the uXRCE-DDS link and
+                         hege_px4_sensors. The first two modes are Gazebo
+                         CLASSIC and this one is not, so they cannot run in the
+                         same simulator - see docs/px4_sitl.md.
+       planar and ros2_control are unaffected by anything in the px4 branches
+       below; the existing simulation keeps running exactly as before. -->
   <xacro:arg name="drive" default="planar"/>
   <xacro:property name="drive" value="$(arg drive)"/>
@@ -159,5 +169,17 @@
     </gazebo>
   </xacro:macro>
-  <link name="base_footprint"/>
+  <link name="base_footprint">
+    <!-- Massless everywhere except px4 mode. There the base_joint below is
+         preserved through SDF conversion, which leaves base_footprint as a
+         real root link, and gz-sim wants a root link to have an inertia. It is
+         1e-4 kg against 1200 kg, so it changes neither the total mass nor the
+         centre of mass in any way that survives rounding. -->
+    <xacro:if value="${drive == 'px4'}">
+      <inertial>
+        <mass value="1e-4"/>
+        <inertia ixx="1e-6" ixy="0" ixz="0" iyy="1e-6" iyz="0" izz="1e-6"/>
+      </inertial>
+    </xacro:if>
+  </link>
   <link name="base_link">
     <visual>
@@ -280,4 +302,10 @@
     <origin xyz="0 0 ${gps_z}" rpy="0 0 0"/>
   </joint>
+  <!-- ============ SENSORS, GAZEBO CLASSIC ============ -->
+  <!-- Wrapped rather than re-indented so the diff against the working
+       simulation stays readable. In px4 mode these are replaced wholesale by
+       the Harmonic sensors further down: the plugin names, the sensor types
+       and the consumer are all different. -->
+  <xacro:unless value="${drive == 'px4'}">
   <!-- ============ IMU SENSOR ============ -->
   <gazebo reference="imu_link">
@@ -338,4 +366,5 @@
     </sensor>
   </gazebo>
+  </xacro:unless>
   <!-- ============ PLANAR DRIVE (keyboard / teleop) ============ -->
   <xacro:if value="${drive == 'planar'}">
@@ -432,3 +461,142 @@
     </gazebo>
   </xacro:if>
+  <!-- ============ PX4 SITL (Gazebo Harmonic) ============ -->
+  <!-- Nothing in this branch talks to ROS. PX4's gz_bridge reads the sensors
+       and writes the joints straight over gz-transport, and everything ROS
+       sees arrives later over uXRCE-DDS via hege_px4_sensors.
+       PX4 finds the sensors by HARDCODED topic paths (GZBridge.cpp):
+         /world/$W/model/$M/link/base_link/sensor/imu_sensor/imu
+         /world/$W/model/$M/link/base_link/sensor/navsat_sensor/navsat
+         /world/$W/model/$M/link/base_link/sensor/magnetometer_sensor/magnetometer
+         /world/$W/model/$M/link/base_link/sensor/air_pressure_sensor/air_pressure
+       So the link name and all four sensor names are fixed by PX4, not chosen
+       by us. Renaming any of them silently gives a vehicle whose EKF2 never
+       receives that sensor. -->
+  <xacro:if value="${drive == 'px4'}">
+    <!-- URDF->SDF conversion lumps a fixed joint's child into its parent.
+         base_link is base_footprint's fixed child, so without this the model
+         would have no link called base_link at all and PX4 would subscribe to
+         four topics that never exist. -->
+    <gazebo reference="base_joint">
+      <preserveFixedJoint>true</preserveFixedJoint>
+    </gazebo>
+    <!-- All four sensors live on base_link because PX4 demands it, and carry
+         the measured lever arms as an explicit pose instead. imu_link and
+         gps_link still exist in the URDF, so robot_state_publisher keeps
+         publishing their TF for navsat_transform and RViz; they simply are not
+         where the simulated hardware is mounted. -->
+    <gazebo reference="base_link">
+      <!-- 1.20 m above the ground = imu_z above base_link. -->
+      <sensor name="imu_sensor" type="imu">
+        <pose>0 0 ${imu_z} 0 0 0</pose>
+        <always_on>1</always_on>
+        <update_rate>250</update_rate>
+        <imu>
+          <angular_velocity>
+            <x><noise type="gaussian"><mean>0.0</mean><stddev>${imu_gyro_noise}</stddev><bias_mean>${imu_gyro_bias}</bias_mean><bias_stddev>${imu_gyro_bias}</bias_stddev></noise></x>
+            <y><noise type="gaussian"><mean>0.0</mean><stddev>${imu_gyro_noise}</stddev><bias_mean>${imu_gyro_bias}</bias_mean><bias_stddev>${imu_gyro_bias}</bias_stddev></noise></y>
+            <z><noise type="gaussian"><mean>0.0</mean><stddev>${imu_gyro_noise}</stddev><bias_mean>${imu_gyro_bias}</bias_mean><bias_stddev>${imu_gyro_bias}</bias_stddev></noise></z>
+          </angular_velocity>
+          <linear_acceleration>
+            <x><noise type="gaussian"><mean>0.0</mean><stddev>${imu_accel_noise}</stddev><bias_mean>${imu_accel_bias}</bias_mean><bias_stddev>${imu_accel_bias}</bias_stddev></noise></x>
+            <y><noise type="gaussian"><mean>0.0</mean><stddev>${imu_accel_noise}</stddev><bias_mean>${imu_accel_bias}</bias_mean><bias_stddev>${imu_accel_bias}</bias_stddev></noise></y>
+            <z><noise type="gaussian"><mean>0.0</mean><stddev>${imu_accel_noise}</stddev><bias_mean>${imu_accel_bias}</bias_mean><bias_stddev>${imu_accel_bias}</bias_stddev></noise></z>
+          </linear_acceleration>
+        </imu>
+      </sensor>
+      <!-- 1.30 m above the ground = gps_z above base_link. Deliberately
+           noiseless: PX4 adds its own GNSS error model through the SIM_GPS_*
+           parameters, and stacking ours on top would make the fix worse than
+           either model describes. gps_noise in this file drives the Gazebo
+           Classic receiver only. -->
+      <sensor name="navsat_sensor" type="navsat">
+        <pose>0 0 ${gps_z} 0 0 0</pose>
+        <always_on>1</always_on>
+        <update_rate>10</update_rate>
+      </sensor>
+      <!-- Neither sensor exists on the real Hege as a separate unit, but EKF2
+           expects both. Noise figures are PX4's own, taken from the stock
+           rover model: they describe the chips, not the vehicle. -->
+      <sensor name="magnetometer_sensor" type="magnetometer">
+        <always_on>1</always_on>
+        <update_rate>100</update_rate>
+        <magnetometer>
+          <x><noise type="gaussian"><stddev>0.0001</stddev></noise></x>
+          <y><noise type="gaussian"><stddev>0.0001</stddev></noise></y>
+          <z><noise type="gaussian"><stddev>0.0001</stddev></noise></z>
+        </magnetometer>
+      </sensor>
+      <sensor name="air_pressure_sensor" type="air_pressure">
+        <always_on>1</always_on>
+        <update_rate>50</update_rate>
+        <air_pressure>
+          <pressure><noise type="gaussian"><mean>0</mean><stddev>3</stddev></noise></pressure>
+        </air_pressure>
+      </sensor>
+    </gazebo>
+    <!-- Traction: the two rear wheels.
+         PX4 sends a gz Actuators message on command/motor_speed and the
+         velocity it carries is (mixer output - 100), so the joint is commanded
+         in rad/s directly. Both rear wheels read actuator 0, which is what
+         makes them a single rigid axle rather than a differential.
+         Hege is rear-wheel drive; PX4's own rover model drives all four. The
+         front wheels below stay free-rolling, which is what the real machine
+         does. -->
+    <gazebo>
+      <plugin filename="gz-sim-joint-controller-system" name="gz::sim::systems::JointController">
+        <joint_name>left_rear_wheel_joint</joint_name>
+        <sub_topic>command/motor_speed</sub_topic>
+        <control_type>velocity</control_type>
+        <use_actuator_msg>true</use_actuator_msg>
+        <actuator_number>0</actuator_number>
+      </plugin>
+    </gazebo>
+    <gazebo>
+      <plugin filename="gz-sim-joint-controller-system" name="gz::sim::systems::JointController">
+        <joint_name>right_rear_wheel_joint</joint_name>
+        <sub_topic>command/motor_speed</sub_topic>
+        <control_type>velocity</control_type>
+        <use_actuator_msg>true</use_actuator_msg>
+        <actuator_number>0</actuator_number>
+      </plugin>
+    </gazebo>
+    <!-- Steering: both front knuckles.
+         PX4 has one steering output, so both sides receive the same angle.
+         That is parallel steering, not true Ackermann geometry - the inner and
+         outer wheels should differ - but it is exactly what PX4's own rover
+         model does, and the error is small at the turning radii this vehicle
+         can reach. The gains are PX4's; raise them if the steering visibly
+         lags the commanded angle on a 1200 kg vehicle. -->
+    <gazebo>
+      <plugin filename="gz-sim-joint-position-controller-system" name="gz::sim::systems::JointPositionController">
+        <joint_name>left_steer_joint</joint_name>
+        <sub_topic>servo_0</sub_topic>
+        <p_gain>100</p_gain>
+        <i_gain>10</i_gain>
+        <d_gain>0</d_gain>
+      </plugin>
+    </gazebo>
+    <gazebo>
+      <plugin filename="gz-sim-joint-position-controller-system" name="gz::sim::systems::JointPositionController">
+        <joint_name>right_steer_joint</joint_name>
+        <sub_topic>servo_0</sub_topic>
+        <p_gain>100</p_gain>
+        <i_gain>10</i_gain>
+        <d_gain>0</d_gain>
+      </plugin>
+    </gazebo>
+    <!-- Publishes joint state on gz-transport only. It is not the ROS
+         /joint_states topic and nothing in the ROS stack consumes it; it is
+         here because it makes the model inspectable from `gz topic`. -->
+    <gazebo>
+      <plugin filename="gz-sim-joint-state-publisher-system" name="gz::sim::systems::JointStatePublisher">
+        <joint_name>left_rear_wheel_joint</joint_name>
+        <joint_name>right_rear_wheel_joint</joint_name>
+        <joint_name>left_steer_joint</joint_name>
+        <joint_name>right_steer_joint</joint_name>
+        <joint_name>left_front_wheel_joint</joint_name>
+        <joint_name>right_front_wheel_joint</joint_name>
+      </plugin>
+    </gazebo>
+  </xacro:if>
 </robot>

Commit message: Adopt oguzissik's vehicle measurements
The two repositories disagreed about the machine itself and both sets were
described as measured. This takes the VERIFIED MEASUREMENTS block from
oguzissik/hege_gps_navigation wholesale, so there is one answer:

    wheelbase           1.91 -> 1.90 m
    rear track          1.50 -> 1.55 m
    front wheel radius  0.27 -> 0.28 m
    max steering        0.600 -> 0.611 rad (35 deg)
    total mass          1200 -> 1300 kg

The numbers appear in five places that cannot see each other, and all of
them moved together: the xacro, controllers.yaml, the PX4 airframe, both
bridge configs and the Nav2 hints. So did everything derived from them -
the geometric turning radius from 2.79 m to 2.71, the airframe's steering
limit in degrees, its yaw rate ceiling from 60 to 63 deg/s, and the prose
in the docs. The Nav2 footprint happens to round to the same polygon, and
its comment now shows the new arithmetic rather than the old.

Two things deliberately not changed. The wheel and knuckle masses stay at
80/45/15 kg: they are estimates in both repositories rather than
measurements, and ours were picked so the mass ratio across a joint does
not make the solver diverge. Only the 1300 kg total is measured and the
chassis absorbs the difference. And minimum_turning_radius stays at 6.0 m,
because it is a measured figure, not a derived one.

That last point is the caveat worth carrying: the radii Nav2 is tuned
against - 4.20 m at 0.6 m/s, 4.64 at 1.0, 5.44 at 1.5 - were measured
before this change. nav2_params.yaml and the README now say so and ask for
a re-measure.

One inconsistency survives and belongs to the upstream repository, not to
us: its xacro says 1.90 m and its bridge_real.yaml says 1.91, and its
README gives the range. This repository uses 1.90 everywhere and the
README says why.

Verified: all four drive modes expand, the generated model carries the new
axle positions and steering limits, every derived number recomputes to
what the files claim, 141 tests pass.

File: src/hege_description/urdf/hege.urdf.xacro (robot description, xacro)
@@ -64,9 +64,9 @@
   <xacro:property name="base_width"    value="1.4"/>
   <xacro:property name="base_height"   value="0.8"/>
-  <!-- Mass. The real machine is 1200 kg. Wheel and knuckle masses are
+  <!-- Mass. The real machine is 1300 kg. Wheel and knuckle masses are
        estimates for tractor-style wheels; the chassis takes whatever is left,
        so the total always comes out at total_mass no matter which of these is
        edited. -->
-  <xacro:property name="total_mass"        value="1200.0"/>
+  <xacro:property name="total_mass"        value="1300.0"/>
   <xacro:property name="rear_wheel_mass"   value="80.0"/>
   <xacro:property name="front_wheel_mass"  value="45.0"/>
@@ -97,19 +97,20 @@
   <xacro:property name="body_z_offset" value="0.4"/>
   <xacro:property name="base_z"        value="1.10"/>
-  <!-- Front and rear wheels are DIFFERENT sizes on Hege: 27 cm front, 40 cm
+  <!-- Front and rear wheels are DIFFERENT sizes on Hege: 28 cm front, 40 cm
        rear. Everything downstream has to respect that - the axle heights below
        are derived from each radius so both pairs touch the ground, and
        controllers.yaml carries the two radii separately. -->
-  <xacro:property name="front_wheel_radius" value="0.27"/>
+  <xacro:property name="front_wheel_radius" value="0.28"/>
   <xacro:property name="rear_wheel_radius"  value="0.40"/>
   <xacro:property name="wheel_width"        value="0.2"/>
-  <!-- Front and rear tracks also differ slightly. -->
-  <xacro:property name="wheelbase"   value="1.91"/>
+  <!-- Front and rear tracks are equal; the wheel sizes are what differ. -->
+  <xacro:property name="wheelbase"   value="1.90"/>
   <xacro:property name="front_track" value="1.55"/>
-  <xacro:property name="rear_track"  value="1.50"/>
-  <!-- STILL UNMEASURED. Minimum turning radius is wheelbase/tan(max_steer),
-       so at 1.91 m wheelbase this value sets it to 2.79 m - nearly three times
-       the old placeholder geometry. Nav2's controller tuning depends on it. -->
-  <xacro:property name="max_steer" value="0.6"/>   <!-- ~34 deg -->
+  <xacro:property name="rear_track"  value="1.55"/>
+  <!-- Minimum turning radius is wheelbase/tan(max_steer), so at 1.90 m
+       wheelbase this sets it to 2.71 m. Nav2's controller tuning depends on
+       it - though Nav2 is held to 6.0 m, which is what the rover was measured
+       to actually achieve once tyre slip is in play. -->
+  <xacro:property name="max_steer" value="0.610865238"/>   <!-- 35 deg -->
   <!-- Axle heights relative to base_link, derived so each wheel rests on the
        ground given its own radius. -->
@@ -168,5 +169,5 @@
       <mu2>1.0</mu2>
       <!-- Contact stiffness and damping, scaled with the vehicle. At the
-           1e6 that suited a 15 kg model, 1200 kg pushes the wheels into the
+           1e6 that suited a 15 kg model, 1300 kg pushes the wheels into the
            ground far enough to change the effective radius and therefore the
            odometry. -->
@@ -181,5 +182,5 @@
          preserved through SDF conversion, which leaves base_footprint as a
          real root link, and gz-sim wants a root link to have an inertia. It is
-         1e-4 kg against 1200 kg, so it changes neither the total mass nor the
+         1e-4 kg against 1300 kg, so it changes neither the total mass nor the
          centre of mass in any way that survives rounding. -->
     <xacro:if value="${drive == 'px4'}">
@@ -253,5 +254,5 @@
       <axis xyz="0 0 1"/>
       <!-- Effort scaled with the vehicle. 100 Nm, sized for the old 15 kg
-           placeholder, cannot turn the front axle of a 1200 kg machine against
+           placeholder, cannot turn the front axle of a 1300 kg machine against
            tyre scrub; the steering simply would not reach its commanded angle.
            Velocity limited to roughly lock to lock in a second and a half,
@@ -680,5 +681,5 @@
          model does, and the error is small at the turning radii this vehicle
          can reach. The gains are PX4's; raise them if the steering visibly
-         lags the commanded angle on a 1200 kg vehicle. -->
+         lags the commanded angle on a 1300 kg vehicle. -->
     <gazebo>
       <plugin filename="gz-sim-joint-position-controller-system" name="gz::sim::systems::JointPositionController">
