Commit message: Fix the Harmonic GPS noise units, and test for them
Gazebo Classic's <gps> sensor takes horizontal position noise in metres.
Harmonic's <navsat> does not: gz-sensors8 applies the value straight to
Latitude().Degree() and Longitude().Degree(), so it is in degrees. The
Harmonic port carried gps_noise across unchanged, which asked for 0.02
degrees of error - 2.2 km. Nothing warns. The fix would simply have been
noise, and the first person to run that simulation would have spent a day
looking at the EKF.

Found by Oguzhan Enes Isik in oguzissik/hege_gps_navigation. The gz branch
now divides by metres_per_latitude_degree; the Classic branch is untouched,
because its units were right.

Two things follow from the same fact. Equal angular noise on the two axes
is not equal metric noise, since one degree of longitude is cos(latitude)
fewer metres than one of latitude - about 0.61 of it here. And Gazebo
publishes the fix with no covariance at all, which navsat_transform
carries into /odometry/gps and the global EKF then uses to decide how far
to move towards each fix. So the bridge now goes to /gps/fix_raw and
sim_gps_covariance.py republishes on /gps/fix with the covariance the
noise settings imply, anisotropy included.

Whether the Classic sensor has the same covariance gap is not established
and the docs say so rather than guess.

hege_description/test/ is new and is the part worth keeping. The model has
four drive modes sharing one file and every way it goes wrong is quiet: a
plugin leaking between simulator generations, base_link vanishing from the
px4 model through fixed-joint lumping, two publishers on the odom edge.
Fourteen tests, no ROS and no Gazebo needed. Reintroducing the units bug
fails two of them, which is how they were checked.

Three of Oguzhan's later changes are deliberately not adopted, with the
reasons in the README: base_footprint moved to the rear axle, which would
mean re-deriving Nav2's footprint and robot_base_frame; lateral friction
lowered to 0.8, which moves the turning radius that is already pending a
re-measure; and a GPS noise evaluator that overlaps what
localization_monitor already does.

File: src/hege_description/urdf/hege.urdf.xacro (robot description, xacro)
@@ -44,4 +44,18 @@
        route, and read the error off the localization monitor. -->
   <xacro:property name="gps_noise" value="0.02"/>
+  <!-- UNITS TRAP. Gazebo Classic's <gps> sensor takes horizontal noise in
+       METRES. Gazebo Harmonic's <navsat> sensor does not: gz-sensors8 applies
+       the value straight to Latitude().Degree() and Longitude().Degree(), so
+       it is in DEGREES. Feeding gps_noise to it unconverted asks for 0.02
+       degrees of error, which is 2.2 km - and nothing warns, the fix just
+       becomes noise. The gz branch below divides by this; the Classic branch
+       must not.
+       Found by Oguzhan Enes Isik in oguzissik/hege_gps_navigation.
+       A consequence worth knowing: the same ANGULAR noise on both axes is not
+       the same METRIC noise, because one degree of longitude is cos(latitude)
+       fewer metres than one of latitude. At this site that makes the east
+       error about 0.61 of the north one. sim_gps_covariance.py carries that
+       into the covariance it publishes. -->
+  <xacro:property name="metres_per_latitude_degree" value="111195.0"/>
   <!-- Gyro and accelerometer bias. A real MEMS IMU's dominant error is not
        white noise but a bias drawn at startup that then wanders, and that is
@@ -431,7 +445,12 @@
         <navsat>
           <position_sensing>
+            <!-- DEGREES here, not metres - see metres_per_latitude_degree at
+                 the top of this file. The Classic sensor above takes the same
+                 quantity in metres, which is exactly what makes this easy to
+                 get wrong. -->
             <horizontal>
-              <noise type="gaussian"><mean>0.0</mean><stddev>${gps_noise}</stddev></noise>
+              <noise type="gaussian"><mean>0.0</mean><stddev>${gps_noise / metres_per_latitude_degree}</stddev></noise>
             </horizontal>
+            <!-- Vertical noise IS in metres, in both simulators. -->
             <vertical>
               <noise type="gaussian"><mean>0.0</mean><stddev>${gps_noise * 2}</stddev></noise>

Commit message: Adopt the last three changes from oguzissik
All three were held back last time for the reasons the README gave. Taking
them means moving what they were measured against, so each one dragged
something with it.

base_footprint moves to the rear axle. That is the bicycle model's
reference point and what ackermann_steering_controller computes odometry
about, so base_frame_id: base_footprint only means what it says with the
frame there. Nav2's footprint polygon is defined about that frame and had
to be re-derived: it now runs from -0.5 m to +2.2 m rather than -1.4 to
+1.3, almost entirely ahead of the origin, which is what a rear-axle
origin looks like.

Lateral tyre friction drops from 1.0 to 0.8, and both friction figures
become named properties instead of literals - lateral grip is the knob
behind the gap between the 2.71 m geometric turning radius and the larger
one the rover drives, so it deserves a name.

hege_evaluation comes in whole. sim_gps_covariance is the part that is not
optional: Gazebo publishes the fix with no covariance at all, and
navsat_transform hands that straight to the global EKF, which then has to
guess how far to move towards each fix. gps_noise_evaluator is the
measuring instrument for the units bug fixed in the last commit - it
scores the fix against ground truth, which is how you learn the GPS is not
the error you configured. sim_gps_covariance moved out of hege_description
into it, matching the upstream layout, and the ground truth topic is now
/hege/ground_truth/odom so both repositories name it the same thing.

The turning radii in nav2_params.yaml are pushed in both directions by
this: lower friction widens the circle, a rear-axle origin narrows it by
about 0.1 m at these radii. 6.0 m still has margin over the arithmetic,
but the comment there now lists all three reasons a re-measure is owed
rather than the one it listed before.

Two new tests pin the frame and the friction properties down, since both
are now load-bearing for numbers elsewhere. 159 tests pass: 141 bridge and
sensor, 16 model, 2 geodesy.

File: src/hege_description/urdf/hege.urdf.xacro (robot description, xacro)
@@ -118,4 +118,10 @@
   <xacro:property name="rear_wheel_radius"  value="0.40"/>
   <xacro:property name="wheel_width"        value="0.2"/>
+  <!-- Tyre friction, longitudinal and lateral. The lateral one is the more
+       interesting of the two: it sets how far the tyres scrub sideways in a
+       corner, which is the whole difference between the 2.71 m geometric
+       turning radius and the larger one the rover actually drives. -->
+  <xacro:property name="wheel_mu_longitudinal" value="0.8"/>
+  <xacro:property name="wheel_mu_lateral"      value="0.8"/>
   <!-- Front and rear tracks are equal; the wheel sizes are what differ. -->
   <xacro:property name="wheelbase"   value="1.90"/>
@@ -179,7 +185,13 @@
     <gazebo reference="${link}">
       <!-- Friction. Tractor tyres on soil, and this is the knob behind the
-           rover turning less sharply than commanded. -->
-      <mu1>1.0</mu1>
-      <mu2>1.0</mu2>
+           rover turning less sharply than commanded: lateral grip is what
+           decides how much the tyres scrub in a corner, and therefore how much
+           wider the achieved circle is than the geometric one.
+           Both 0.8, matching oguzissik/hege_gps_navigation. They were 1.0/1.0
+           here, and the measured radii in nav2_params.yaml come from that -
+           lowering lateral grip widens the circle, so those numbers are now
+           pending a re-measure. -->
+      <mu1>${wheel_mu_longitudinal}</mu1>
+      <mu2>${wheel_mu_lateral}</mu2>
       <!-- Contact stiffness and damping, scaled with the vehicle. At the
            1e6 that suited a 15 kg model, 1300 kg pushes the wheels into the
@@ -218,8 +230,20 @@
                        cx="${base_com_x}" cz="${base_com_z}"/>
   </link>
+  <!-- base_footprint sits at the REAR AXLE, on the ground - not under the
+       middle of the vehicle. base_link is therefore wheelbase/2 forward of it.
+       The rear axle is the reference point of the bicycle model, and it is the
+       point ackermann_steering_controller computes its odometry about, so
+       base_frame_id: base_footprint only means what it says with the frame
+       here. Following oguzissik/hege_gps_navigation.
+       Two things downstream are defined about this frame and had to move with
+       it: Nav2's footprint polygon in nav2_params.yaml, which is now measured
+       from the rear axle rather than the centre, and the turning radii in the
+       same file - a circle traced by the rear axle is smaller than the one
+       traced by the vehicle centre by sqrt(R^2 + (L/2)^2) - R, about 0.1 m at
+       these radii. -->
   <joint name="base_joint" type="fixed">
     <parent link="base_footprint"/>
     <child  link="base_link"/>
-    <origin xyz="0 0 ${base_z}"/>
+    <origin xyz="${wheelbase/2} 0 ${base_z}"/>
   </joint>
   <!-- ============ REAR (driven) WHEELS ============ -->
@@ -472,6 +496,6 @@
         <odom_frame>world</odom_frame>
         <robot_base_frame>base_footprint</robot_base_frame>
-        <odom_topic>/ground_truth/odom</odom_topic>
-        <tf_topic>/ground_truth/tf_unused</tf_topic>
+        <odom_topic>/hege/ground_truth/odom</odom_topic>
+        <tf_topic>/hege/ground_truth/pose</tf_topic>
         <odom_publish_frequency>50</odom_publish_frequency>
         <dimensions>3</dimensions>
